File: kicad/8080_ECB_SBC/IO_PIC.kicad_sch (KiCad schematic)
At the start: 38 parts, among them J2 SPEAKER, J3 Conn_01x07, J4 RS232, Q2 PN2222A, U17 74LS390, U18 8253, U19 8259A, U20 8251, U21 MAX232, U22 74HC374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

Commit message: cleanup
Parts:
- C22, C23, C24, C25: Mfr. No FK28X5R1E105K -> FG28X7R1E105KRT06
- R5: Mfr. No CF18JT1R00 -> OJ10G5E-R52
